File: ProjectFolder/LEDCubeBufferDemux.sch (KiCad schematic (older format))
At the start: 12 parts, among them U1 SN74LVC1G139DCTR, U2 SN74LVC1G139DCTR, U3 SN74LVC1G139DCTR, U4 ULN2003ADR, U5 ULN2003ADR, U6 SN74LVC1G139DCTR

Commit message: Mostly finished PCB layout
Connections:
- net +5V: now also U4.7 (7B); no longer U4.4 (4B)
- net S1Y1: now also U4.4 (4B); no longer U4.1 (1B)
- net S1Y2: now also U4.5 (5B); no longer U4.2 (2B)
- net S1Y3: now also U4.6 (6B); no longer U4.3 (3B)
- net S2Y1: now also U4.1 (1B); no longer U4.5 (5B)
- net S2Y2: now also U4.2 (2B); no longer U4.6 (6B)
- net S2Y3: now also U4.3 (3B); no longer U4.7 (7B)
- net Slice1Cathode1: now also U4.13 (4C); no longer U4.16 (1C)
- net Slice1Cathode2: now also U4.12 (5C); no longer U4.15 (2C)
- net Slice1Cathode3: now also U4.11 (6C); no longer U4.14 (3C)
- net Slice2Cathode1: now also U4.16 (1C); no longer U4.12 (5C)
- net Slice2Cathode2: now also U4.15 (2C); no longer U4.11 (6C)
- net Slice2Cathode3: now also U4.14 (3C); no longer U4.10 (7C)
Other:
- moved on the sheet: U1, U2
Changed lines of the file:
@@
 Comment4 "PCB Designer: Donovan Squires"
 $EndDescr
+Text HLabel 2250 3100 0    60   Input ~ 0
+Slice1EN
 Text HLabel 2250 1900 0    60   Input ~ 0
-Slice1EN
-Text HLabel 2250 3100 0    60   Input ~ 0
 Slice2EN
 Text HLabel 2250 4400 0    60   Input ~ 0
@@
 Text HLabel 7700 3900 0    60   Input ~ 0
 AnodeB
+Text HLabel 5950 2800 2    60   Output ~ 0
+Slice1Cathode3
+Text HLabel 5950 2700 2    60   Output ~ 0
+Slice1Cathode2
+Text HLabel 5950 2600 2    60   Output ~ 0
+Slice1Cathode1
 Text HLabel 5950 2500 2    60   Output ~ 0
-Slice1Cathode3
+Slice2Cathode3
 Text HLabel 5950 2400 2    60   Output ~ 0
-Slice1Cathode2
+Slice2Cathode2
 Text HLabel 5950 2300 2    60   Output ~ 0
-Slice1Cathode1
-Text HLabel 5950 2900 2    60   Output ~ 0
-Slice2Cathode3
-Text HLabel 5950 2800 2    60   Output ~ 0
-Slice2Cathode2
-Text HLabel 5950 2700 2    60   Output ~ 0
 Slice2Cathode1
 Text HLabel 5950 4800 2    60   Output ~ 0
@@
 L SN74LVC1G139DCTR U1
 U 1 1 550AC020
-P 2950 2150
-F 0 "U1" H 2700 2550 60  0000 L CNN
-F 1 "SN74LVC1G139DCTR" H 2700 1750 60  0000 L CNN
-F 2 "sn74lvc1g139dctr:sn74lvc1g139dctr" H 3050 2000 60  0001 C CNN
-F 3 "" H 3050 2000 60  0000 C CNN
-F 4 "Texas Instruments" H 2950 2150 60  0001 C CNN "Manufacturer"
-F 5 "SN74LVC1G139DCTR" H 2950 2150 60  0001 C CNN "Manufacturer Part Number"
-F 6 "Digi-Key" H 2950 2150 60  0001 C CNN "Supplier"
-F 7 "296-18235-1-ND" H 2950 2150 60  0001 C CNN "Supplier Part Number"
-	1    2950 2150
+P 2950 3350
+F 0 "U1" H 2700 3750 60  0000 L CNN
+F 1 "SN74LVC1G139DCTR" H 2700 2950 60  0000 L CNN
+F 2 "sn74lvc1g139dctr:sn74lvc1g139dctr" H 3050 3200 60  0001 C CNN
+F 3 "" H 3050 3200 60  0000 C CNN
+F 4 "Texas Instruments" H 2950 3350 60  0001 C CNN "Manufacturer"
+F 5 "SN74LVC1G139DCTR" H 2950 3350 60  0001 C CNN "Manufacturer Part Number"
+F 6 "Digi-Key" H 2950 3350 60  0001 C CNN "Supplier"
+F 7 "296-18235-1-ND" H 2950 3350 60  0001 C CNN "Supplier Part Number"
+	1    2950 3350
 	1    0    0    -1
 $EndComp
@@
 Connection ~ 1350 3400
 Wire Wire Line
+	4000 2100 4000 2300
+Wire Wire Line
+	4000 2300 4450 2300
+Wire Wire Line
+	4450 2400 3900 2400
+Wire Wire Line
+	3900 2400 3900 2200
+Wire Wire Line
+	3900 3400 3400 3400
+Wire Wire Line
+	3400 3500 4000 3500
+Wire Wire Line
+	3800 2300 3800 2500
+Wire Wire Line
+	3800 2500 4450 2500
+Wire Wire Line
 	3400 2100 4000 2100
 Wire Wire Line
-	4000 2100 4000 2300
-Wire Wire Line
-	4000 2300 4450 2300
-Wire Wire Line
-	4450 2400 3900 2400
-Wire Wire Line
-	3900 2400 3900 2200
+	3800 2600 3800 3300
 Wire Wire Line
 	3900 2200 3400 2200
 Wire Wire Line
-	3400 2300 3800 2300
-Wire Wire Line
-	3800 2300 3800 2500
-Wire Wire Line
-	3800 2500 4450 2500
-Wire Wire Line
-	3800 3300 3400 3300
-Wire Wire Line
-	3800 2700 3800 3300
-Wire Wire Line
-	3900 3400 3400 3400
-Wire Wire Line
-	3900 2800 3900 3400
-Wire Wire Line
-	4000 2900 4000 3500
-Wire Wire Line
-	4000 3500 3400 3500
+	3900 2700 3900 3400
+Wire Wire Line
+	4000 3500 4000 2800
 Wire Wire Line
 	4450 3100 4350 3100
@@
 Leave unused ouputs\nunconnected
 Wire Wire Line
+	5450 2600 5950 2600
+Wire Wire Line
+	5450 2700 5950 2700
+Wire Wire Line
+	5450 2800 5950 2800
+Wire Wire Line
 	5450 2300 5950 2300
 Wire Wire Line
@@
 Wire Wire Line
 	5450 2500 5950 2500
-Wire Wire Line
-	5450 2700 5950 2700
-Wire Wire Line
-	5450 2800 5950 2800
-Wire Wire Line
-	5450 2900 5950 2900
 Wire Wire Line
 	5450 4800 5950 4800
@@
 NoConn ~ 5450 5100
 NoConn ~ 5450 5200
-NoConn ~ 5450 2600
+NoConn ~ 5450 2900
 NoConn ~ 3400 2000
 NoConn ~ 3400 3200
@@
 Text Notes 2750 6950 0    60   ~ 0
 Place decoupling capacitors\nclose to E pins
+Text Label 3550 3300 0    60   ~ 0
+S1Y1
+Text Label 3550 3400 0    60   ~ 0
+S1Y2
+Text Label 3550 3500 0    60   ~ 0
+S1Y3
 Text Label 3550 2100 0    60   ~ 0
-S1Y1
+S2Y1
 Text Label 3550 2200 0    60   ~ 0
-S1Y2
+S2Y2
 Text Label 3550 2300 0    60   ~ 0
-S1Y3
-Text Label 3550 3300 0    60   ~ 0
-S2Y1
-Text Label 3550 3400 0    60   ~ 0
-S2Y2
-Text Label 3550 3500 0    60   ~ 0
 S2Y3
 Text Label 3550 4600 0    60   ~ 0
@@
 $EndComp
 Wire Wire Line
-	4450 2700 3800 2700
-Wire Wire Line
-	4450 2800 3900 2800
-Wire Wire Line
-	4450 2900 4000 2900
-Wire Wire Line
 	4350 3100 4350 5650
 Wire Wire Line
-	4250 2600 4450 2600
-Wire Wire Line
 	4250 4900 4450 4900
-Connection ~ 4250 2600
 Wire Wire Line
 	4250 5000 4450 5000
@@
 L SN74LVC1G139DCTR U2
 U 1 1 550B6026
-P 2950 3350
-F 0 "U2" H 2700 3750 60  0000 L CNN
-F 1 "SN74LVC1G139DCTR" H 2700 2950 60  0000 L CNN
-F 2 "sn74lvc1g139dctr:sn74lvc1g139dctr" H 3050 3200 60  0001 C CNN
-F 3 "" H 3050 3200 60  0000 C CNN
-F 4 "Texas Instruments" H 2950 3350 60  0001 C CNN "Manufacturer"
-F 5 "SN74LVC1G139DCTR" H 2950 3350 60  0001 C CNN "Manufacturer Part Number"
-F 6 "Digi-Key" H 2950 3350 60  0001 C CNN "Supplier"
-F 7 "296-18235-1-ND" H 2950 3350 60  0001 C CNN "Supplier Part Number"
-	1    2950 3350
+P 2950 2150
+F 0 "U2" H 2700 2550 60  0000 L CNN
+F 1 "SN74LVC1G139DCTR" H 2700 1750 60  0000 L CNN
+F 2 "sn74lvc1g139dctr:sn74lvc1g139dctr" H 3050 2000 60  0001 C CNN
+F 3 "" H 3050 2000 60  0000 C CNN
+F 4 "Texas Instruments" H 2950 2150 60  0001 C CNN "Manufacturer"
+F 5 "SN74LVC1G139DCTR" H 2950 2150 60  0001 C CNN "Manufacturer Part Number"
+F 6 "Digi-Key" H 2950 2150 60  0001 C CNN "Supplier"
+F 7 "296-18235-1-ND" H 2950 2150 60  0001 C CNN "Supplier Part Number"
+	1    2950 2150
 	1    0    0    -1
 $EndComp
@@
 	1    0    0    -1
 $EndComp
+Wire Wire Line
+	3800 2600 4450 2600
+Wire Wire Line
+	4450 2700 3900 2700
+Wire Wire Line
+	4000 2800 4450 2800
+Wire Wire Line
+	4250 2900 4450 2900
+Connection ~ 4250 2900
+Wire Wire Line
+	3400 2300 3800 2300
+Wire Wire Line
+	3800 3300 3400 3300
 $EndSCHEMATC
